File: Claculator_Keypad/Claculator_Keypad.kicad_pcb (KiCad board)
At the start: 2 copper layers, 198 parts, among them J1 Conn_01x15_Pin, J3 Conn_01x15_Pin, SW1 SW_Push, SW10 SW_Push, SW11 SW_Push, SW12 SW_Push, SW13 SW_Push, SW14 SW_Push, SW15 SW_Push, SW16 SW_Push, SW17 SW_Push, SW18 SW_Push, SW19 SW_Push, SW2 SW_Push, SW20 SW_Push, SW21 SW_Push, SW22 SW_Push, SW23 SW_Push, SW24 SW_Push, SW25 SW_Push, SW26 SW_Push, SW27 SW_Push, SW28 SW_Push, SW29 SW_Push, SW3 SW_Push, SW30 SW_Push, SW31 SW_Push, SW32 SW_Push, SW33 SW_Push, SW34 SW_Push, SW35 SW_Push, SW36 SW_Push, SW37 SW_Push, SW38 SW_Push, SW39 SW_Push, SW4 SW_Push, SW40 SW_Push, SW41 SW_Push, SW42 SW_Push, SW43 SW_Push, SW44 SW_Push, SW45 SW_Push, SW46 SW_Push, SW47 SW_Push, SW48 SW_Push, SW5 SW_Push, SW6 SW_Push, SW7 SW_Push, SW8 SW_Push, SW9 SW_Push, U1 74HC154, U12 74HC7541, U16 74HC541, U17 74HC541, U18 74HC7541, U2 74HC4024, U20 74HC7541, U22 74HC7541, U24 74HC541, U25 74HC7541, U27 74HC7541, U3 NE555D, U4 74HC14, U5 74HC00

Commit message: Not sure
Parts:
- removed C25, C26, C36, C37, C46, C47, C56, C57, C66, C67, C68, C69, C70, C73, C74, C79, C80, C81, C82: 1uF, Capacitor_SMD:C_1206_3216Metric
- removed R45, R46, R47, R48, R49, R50: 4.7k, Resistor_SMD:R_1206_3216Metric
- removed SW41, SW42, SW43, SW44, SW45, SW46, SW47, SW48: SW_Push, keyswitches:SW_MX
- added D1: D, Package_TO_SOT_SMD:SOT-323_SC-70, B.Cu at (160.7, 49.2)
- added D2: D, Package_TO_SOT_SMD:SOT-323_SC-70, B.Cu at (157.5, 49.2)
- added D3: D, Package_TO_SOT_SMD:SOT-323_SC-70, B.Cu at (154.3, 49.2)
- added D4: D, Package_TO_SOT_SMD:SOT-323_SC-70, B.Cu at (151.2, 49.2)
- added D5: D, Package_TO_SOT_SMD:SOT-323_SC-70, B.Cu at (148.0, 49.2)
- added D6: D, Package_TO_SOT_SMD:SOT-323_SC-70, B.Cu at (97.2, 52.1)
- added G***: LOGO, LOGO, B.Cu at (28.6, 90.2)
- added G***: LOGO, LOGO, B.Cu at (40.6, 92.1)
- added G***: LOGO, LOGO, B.Cu at (61.0, 70.5)
- added G***: LOGO, LOGO, B.Cu at (48.3, 90.2)
- added G***: LOGO, LOGO, B.Cu at (88.3, 92.1)
- added G***: LOGO, LOGO, B.Cu at (68.6, 90.8)
- added G***: LOGO, LOGO, B.Cu at (45.1, 70.5)
- added J2: Conn_01x15_Pin, Connector_PinHeader_2.54mm:PinHeader_1x15_P2.54mm_Vertical, B.Cu at (87.6, 26.7)
- added J4: Conn_01x04_Pin, Connector_PinHeader_2.54mm:PinHeader_1x04_P2.54mm_Vertical, B.Cu at (23.5, 48.1)
- added J5: Conn_01x04_Pin, Connector_PinHeader_2.54mm:PinHeader_1x04_P2.54mm_Vertical, B.Cu at (23.5, 44.3)
- added U10: 74HC86, Package_SO:SOIC-14_3.9x8.7mm_P1.27mm, B.Cu at (95.8, 43.8)
- added U11: 74HC688, Package_SO:SOIC-20W_7.5x12.8mm_P1.27mm, B.Cu at (107.3, 34.9)
- added U13: 74HC08, Package_SO:SOIC-14_3.9x8.7mm_P1.27mm, B.Cu at (87.6, 34.3)
- added U14: 74HC08, Package_SO:SOIC-14_3.9x8.7mm_P1.27mm, B.Cu at (87.6, 43.8)
- added U15: IDT7202, Package_SO:SOIC-28W_7.5x18.7mm_P1.27mm, B.Cu at (54.6, 43.8)
- added U19: CC56-12EWA, Display_7Segment:CA56-12EWA, F.Cu at (144.4, 44.2)
- added U21: 74LS173, Package_SO:SOIC-16_3.9x9.9mm_P1.27mm, B.Cu at (213.4, 36.2)
- added U23: 74LS173, Package_SO:SOIC-16_3.9x9.9mm_P1.27mm, B.Cu at (189.8, 36.2)
- added U26: 74LS173, Package_SO:SOIC-16_3.9x9.9mm_P1.27mm, B.Cu at (181.5, 36.2)
- added U28: 74LS173, Package_SO:SOIC-16_3.9x9.9mm_P1.27mm, B.Cu at (173.3, 36.2)
- added U29: 74LS173, Package_SO:SOIC-16_3.9x9.9mm_P1.27mm, B.Cu at (221.7, 47.0)
- added U30: CC56-12EWA, Display_7Segment:CA56-12EWA, F.Cu at (195.2, 44.2)
- added U31: 74HC86, Package_SO:SOIC-14_3.9x8.7mm_P1.27mm, B.Cu at (104.8, 48.3)
- added U36: 74LS173, Package_SO:SOIC-16_3.9x9.9mm_P1.27mm, B.Cu at (213.4, 47.0)
- added U37: 74LS173, Package_SO:SOIC-16_3.9x9.9mm_P1.27mm, B.Cu at (189.8, 47.0)
- added U38: 74LS173, Package_SO:SOIC-16_3.9x9.9mm_P1.27mm, B.Cu at (181.5, 47.0)
- added U39: 74LS173, Package_SO:SOIC-16_3.9x9.9mm_P1.27mm, B.Cu at (173.3, 47.0)
- added U6: 74HC32, Package_SO:SOIC-14_3.9x8.7mm_P1.27mm, B.Cu at (129.6, 48.3)
- added U7: 74LS173, Package_SO:SOIC-16_3.9x9.9mm_P1.27mm, B.Cu at (221.7, 36.2)
- added U8: 74HC02, Package_SO:SOIC-14_3.9x8.7mm_P1.27mm, B.Cu at (121.2, 48.3)
- added U9: 74HC86, Package_SO:SOIC-14_3.9x8.7mm_P1.27mm, B.Cu at (95.8, 34.3)
- C1, C10, C11, C12, C13, C14, C15, C16, C17, C18, C19, C2, C20, C21, C22, C23, C24, C27, C28, C29, C3, C30, C31, C32, C33, C34, C35, C38, C39, C4, C40, C41, C42, C43, C44, C45, C48, C49, C5, C50, C51, C52, C53, C54, C55, C58, C59, C6, C60, C61, C62, C63, C64, C65, C7, C71, C72, C76, C77, C78, C8, C83, C9: footprint Capacitor_SMD:C_1206_3216Metric -> Capacitor_SMD:C_0805_2012Metric_Pad1.18x1.45mm_HandSolder; moved to B.Cu
- C75: value 1uF -> 1nF; footprint Capacitor_SMD:C_1206_3216Metric -> Capacitor_SMD:C_0805_2012Metric_Pad1.18x1.45mm_HandSolder; moved to B.Cu
- J1, U1, U12, U16, U17, U18, U2, U20, U22, U24, U27, U3, U4, U5: moved to B.Cu
- J3: value Conn_01x15_Pin -> Conn_01x16_Pin; footprint Connector_PinHeader_2.54mm:PinHeader_1x15_P2.54mm_Vertical -> Connector_PinHeader_2.54mm:PinHeader_1x16_P2.54mm_Vertical; moved to B.Cu
- R1, R10, R11, R12, R13, R14, R15, R16, R17, R18, R19, R2, R20, R21, R22, R23, R24, R25, R26, R27, R28, R29, R3, R30, R31, R32, R33, R34, R35, R36, R37, R38, R39, R4, R40, R41, R42, R5, R6, R7, R8, R9: footprint Resistor_SMD:R_1206_3216Metric -> Resistor_SMD:R_0805_2012Metric_Pad1.20x1.40mm_HandSolder; moved to B.Cu
- R43: value 4.7k -> 1k; footprint Resistor_SMD:R_1206_3216Metric -> Resistor_SMD:R_0805_2012Metric_Pad1.20x1.40mm_HandSolder; moved to B.Cu
- R44: value 4.7k -> 10k; footprint Resistor_SMD:R_1206_3216Metric -> Resistor_SMD:R_0805_2012Metric_Pad1.20x1.40mm_HandSolder; moved to B.Cu
- SW1, SW10, SW11, SW12, SW13, SW14, SW15, SW16, SW17, SW18, SW19, SW2, SW20, SW21, SW22, SW23, SW24, SW25, SW26, SW27, SW28, SW29, SW3, SW30, SW31, SW32, SW33, SW34, SW35, SW36, SW37, SW38, SW39, SW4, SW40, SW5, SW6, SW7, SW8, SW9, SW_Rst1: footprint keyswitches:SW_MX -> keyswitches:Kailh_socket_MX
- U25: value 74HC7541 -> 74LS377; moved to B.Cu
- moved SW4 447.4 mm to (218.0, 77.4), turned to 180 degrees
- moved SW2 444.8 mm to (218.0, 57.4), turned to 180 degrees
- moved SW36 431.2 mm to (178.0, 77.4), turned to 180 degrees
- moved SW34 430.2 mm to (177.8, 57.4), turned to 180 degrees
- moved SW5 427.1 mm to (198.0, 97.4), turned to 180 degrees
- moved SW3 424.4 mm to (198.0, 77.4), turned to 180 degrees
- moved SW8 424.0 mm to (218.0, 117.4), turned to 180 degrees
- moved SW6 422.3 mm to (218.0, 97.4), turned to 180 degrees
- moved SW12 422.2 mm to (134.7, 77.4), turned to 180 degrees
- moved SW10 421.4 mm to (134.7, 57.4), turned to 180 degrees
- moved SW38 413.9 mm to (178.0, 97.4), turned to 180 degrees
- moved SW40 413.6 mm to (178.0, 117.4), turned to 180 degrees
- moved SW37 411.0 mm to (158.0, 97.4), turned to 180 degrees
- moved SW35 410.2 mm to (158.0, 77.4), turned to 180 degrees
- moved SW14 404.8 mm to (134.7, 97.4), turned to 180 degrees
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Connections:
- C4 pad 1: Net-(U25-A0) -> +5V
- C75 pad 1: Net-(U25-A3) -> Net-(C75-Pad1)
- C76 pad 1: Net-(U25-A4) -> +5V
- C77 pad 1: Net-(U25-A5) -> +5V
- C78 pad 1: Net-(U25-A6) -> +5V
- J1 pad 10: D3 -> D4
- J1 pad 11: D4 -> D3
- J1 pad 12: D5 -> D2
- J1 pad 13: D6 -> D1
- J1 pad 14: D7 -> D0
- J1 pad 3: WEb -> SelB
- J1 pad 4: SelB -> Phi2
- J1 pad 5: Phi2 -> Rstb
- J1 pad 6: Rstb -> INTb
- J1 pad 7: D0 -> D7
- J1 pad 8: D1 -> D6
- J1 pad 9: D2 -> D5
- J3 pad 1: GND -> 7SEG_A
- J3 pad 10: D3 -> 7SEG_1
- J3 pad 11: D4 -> 7SEG_2
- J3 pad 12: D5 -> 7SEG_3
- J3 pad 13: D6 -> 7SEG_4
- J3 pad 14: D7 -> 7SEG_5
- J3 pad 15: A0 -> 7SEG_6
- J3 pad 2: +5V -> 7SEG_B
- J3 pad 3: WEb -> 7SEG_C
- J3 pad 4: SelB -> 7SEG_D
- J3 pad 5: Phi2 -> 7SEG_E
- J3 pad 6: Rstb -> 7SEG_F
- J3 pad 7: D0 -> 7SEG_G
- J3 pad 8: D1 -> 7SEG_H
- J3 pad 9: D2 -> 7SEG_0
- R43 pad 1: Net-(U25-A0) -> FI_W
- R43 pad 2: GND -> Net-(C75-Pad1)
- R44 pad 1: Net-(U25-A1) -> +5V
- R44 pad 2: GND -> RValidB
- SW_Rst1 pad 1: Rstb -> GND
- SW_Rst1 pad 2: GND -> Rstb
- U1 pad 6: R5b -> unconnected-(U1-~{S5}-Pad6)
- U16 pad 19: Q1 -> Q1b
- U17 pad 1: Q2 -> Q1
- U17 pad 19: Q1b -> Q2b
- U25 pad 1: GND -> Net-(U25-~{E})
- U25 pad 11: C7L -> ROW_CLK
- U25 pad 12: C6L -> C4
- U25 pad 13: C5L -> C4L
- U25 pad 14: C4L -> C5L
- U25 pad 15: C3L -> C5
- U25 pad 16: C2L -> C6
- U25 pad 17: C1L -> C6L
- U25 pad 18: C0L -> C7L
- U25 pad 19: R5b -> C7
- U25 pad 2: Net-(U25-A0) -> C0
- U25 pad 3: Net-(U25-A1) -> C0L
- U25 pad 4: Net-(U25-A2) -> C1L
- U25 pad 5: Net-(U25-A3) -> C1
- U25 pad 6: Net-(U25-A4) -> C2
- U25 pad 7: Net-(U25-A5) -> C2L
- U25 pad 8: Net-(U25-A6) -> C3L
- U25 pad 9: Net-(U25-A7) -> C3
- U4 pad 10: (no net) -> FI_Wb
- U4 pad 11: (no net) -> Net-(C75-Pad1)
- U4 pad 12: (no net) -> Net-(U4-Pad12)
- U4 pad 13: (no net) -> Net-(U11-P=R)
- U4 pad 5: (no net) -> Net-(U4-Pad5)
- U4 pad 6: (no net) -> Net-(U25-~{E})
- U4 pad 8: (no net) -> Net-(U4-Pad8)
- U4 pad 9: (no net) -> CHG
- U5 pad 3: LATCH_WEb -> Net-(U5-Pad3)
- U5 pad 4: unconnected-(U5-Pad4) -> Q0
- U5 pad 5: CHG -> Net-(U31-Pad3)
- U5 pad 6: FI_Wb -> Net-(U5-Pad6)
Routing:
- net GND: track 0.00 -> 414.1 mm, vias 0 -> 363
- net C7L: track 0.00 -> 299.2 mm, vias 0 -> 8
- net C6L: track 0.00 -> 294.9 mm, vias 0 -> 8
- net C5L: track 0.00 -> 287.7 mm, vias 0 -> 7
- net C3L: track 0.00 -> 286.7 mm, vias 0 -> 7
- net C0L: track 0.00 -> 286.2 mm, vias 0 -> 8
- net C1L: track 0.00 -> 285.3 mm, vias 0 -> 8
- net C2L: track 0.00 -> 284.3 mm, vias 0 -> 7
- net C4L: track 0.00 -> 283.2 mm, vias 0 -> 7
- net R4b: track 0.00 -> 269.6 mm, vias 0 -> 5
- net +5V: track 0.00 -> 264.3 mm, vias 0 -> 82
- net R1b: track 0.00 -> 234.5 mm, vias 0 -> 4
- net R3b: track 0.00 -> 233.2 mm, vias 0 -> 5
- net R2b: track 0.00 -> 232.2 mm, vias 0 -> 4
- net ROW_CLK: track 0.00 -> 223.0 mm, vias 0 -> 13
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- added copper zone on In2.Cu, net +5V
- added copper zone on B.Cu, net GND
- added copper zone on F.Cu, net GND
- added copper zone on In1.Cu, net GND
- added copper zone on In3.Cu, net GND
- added copper zone on In4.Cu, net GND
Other:
- board outline added: 210 x 119 mm
- copper layers 2 -> 6
- board text added: "5V"
- board text added: "8x5-Key Keypad Driver"
- board text added: "A"
- board text added: "A 6502 Project"
- board text added: "A0"
- board text added: "B"
- board text added: "By Robbie Mones"
- board text added: "C"
- board text added: "Claculator"
- board text added: "D"
- board text added: "D0"
- board text added: "D1"
- board text added: "D2"
- board text added: "D3"
- board text added: "D4"
- board text added: "D5"
- board text added: "D6"
- board text added: "D7"
- board text added: "Designed and Built by Robbie Mones"
- board text added: "E"
- board text added: "F"
- board text added: "G"
- board text added: "GND"
- board text added: "H"
- board text added: "INTb"
- board text added: "P2"
- board text added: "RSTb"
- board text added: "Rev 1"
- board text added: "Sb"
