File: Claculator_Keypad/extras.kicad_sch (KiCad schematic)
At the start: 23 parts, among them U10 74HC86, U13 74LS08, U14 74LS08, U26 74HC14, U31 74HC86, U4 74HC14, U5 74HC00, U7 74HC02, U8 74HC02, U9 74HC86

Commit message: Not sure
Parts:
- removed C11, C12, C23, C68, C69, C7, C70, C82: 1uF, Capacitor_SMD:C_1206_3216Metric, symbol Device:C_Polarized_Small
- removed U26: 74HC14, symbol 74xx:74HC14
- removed unit 2 of U31
- removed unit 3 of U31
- removed U7: 74HC02, symbol 74xx:74HC02
- added J3: Conn_01x16_Pin, Connector_PinHeader_2.54mm:PinHeader_1x16_P2.54mm_Vertical, symbol Connector:Conn_01x16_Pin
- added J4, J5: Conn_01x04_Pin, Connector_PinHeader_2.54mm:PinHeader_1x04_P2.54mm_Vertical, symbol Connector:Conn_01x04_Pin
- added U19, U30: CC56-12EWA, Display_7Segment:CA56-12EWA, symbol Display_Character:CC56-12EWA
- added U6: 74HC32, Package_SO:SOIC-14_3.9x8.7mm_P1.27mm, symbol Custom:74HCS32
- C24, C6, C8, C9: footprint Capacitor_SMD:C_1206_3216Metric -> Capacitor_SMD:C_0805_2012Metric_Pad1.18x1.45mm_HandSolder
- SW_Rst1: footprint keyswitches:SW_MX -> keyswitches:Kailh_socket_MX
- U10, U31, U8, U9: footprint (none) -> Package_SO:SOIC-14_3.9x8.7mm_P1.27mm
- U13, U14: value 74LS08 -> 74HC08; footprint (none) -> Package_SO:SOIC-14_3.9x8.7mm_P1.27mm
Connections:
- net +5V: now also J4.1 (Pin_1), J4.2 (Pin_2), J4.3 (Pin_3), J4.4 (Pin_4), U6.14 (VCC)
- net GND: now also SW_Rst1.1, U31.12, U31.13, J5.1 (Pin_1), J5.2 (Pin_2), J5.3 (Pin_3), J5.4 (Pin_4), U6.10, U6.12, U6.13, U6.7 (GND), U6.9; no longer SW_Rst1.2
- net Rstb: now also SW_Rst1.2; no longer SW_Rst1.1
- new net 7SEG_0: J3.9 (Pin_9), U19.12 (CC1)
- new net 7SEG_1: J3.10 (Pin_10), U19.9 (CC2)
- new net 7SEG_2: J3.11 (Pin_11), U19.8 (CC3)
- new net 7SEG_3: J3.12 (Pin_12), U19.6 (CC4)
- new net 7SEG_4: J3.13 (Pin_13), U30.12 (CC1)
- new net 7SEG_5: J3.14 (Pin_14), U30.9 (CC2)
- new net 7SEG_6: J3.15 (Pin_15), U30.8 (CC3)
- new net 7SEG_7: J3.16 (Pin_16), U30.6 (CC4)
- new net 7SEG_A: J3.1 (Pin_1), U19.11 (a), U30.11 (a)
- new net 7SEG_B: J3.2 (Pin_2), U19.7 (b), U30.7 (b)
- new net 7SEG_C: J3.3 (Pin_3), U19.4 (c), U30.4 (c)
- new net 7SEG_D: J3.4 (Pin_4), U19.2 (d), U30.2 (d)
- new net 7SEG_E: J3.5 (Pin_5), U19.1 (e), U30.1 (e)
- new net 7SEG_F: J3.6 (Pin_6), U19.10 (f), U30.10 (f)
- new net 7SEG_G: J3.7 (Pin_7), U19.5 (g), U30.5 (g)
- new net 7SEG_H: J3.8 (Pin_8), U19.3 (DPX), U30.3 (DPX)
- no-connect marks 0 -> 3
Other:
- moved on the sheet: C24
