File: Claculator_Keypad/row.kicad_sch (KiCad schematic)
At the start: 29 parts, among them SW1 SW_Push, SW2 SW_Push, SW3 SW_Push, SW4 SW_Push, SW5 SW_Push, SW6 SW_Push, SW7 SW_Push, SW8 SW_Push, U12 74HC7541, U6 74HCT574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

Commit message: Not sure
Parts:
- removed C10, C14: 1uF, Capacitor_SMD:C_1206_3216Metric, symbol Device:C_Polarized_Small
- removed U6: 74HCT574, symbol 74xx:74HCT574
- removed U7: 74HC02, symbol 74xx:74HC02
- added C4, C7: 1uF, Capacitor_SMD:C_0805_2012Metric_Pad1.18x1.45mm_HandSolder, symbol Device:C_Polarized_Small
- added U29, U7: 74LS173, Package_SO:SOIC-16_3.9x9.9mm_P1.27mm, symbol 74xx:74LS173
- C15, C16, C17, C18, C19, C20, C21, C22: footprint Capacitor_SMD:C_1206_3216Metric -> Capacitor_SMD:C_0805_2012Metric_Pad1.18x1.45mm_HandSolder
- R10, R3, R4, R5, R6, R7, R8, R9: footprint Resistor_SMD:R_1206_3216Metric -> Resistor_SMD:R_0805_2012Metric_Pad1.20x1.40mm_HandSolder
- SW1, SW2, SW3, SW4, SW5, SW6, SW7, SW8: footprint keyswitches:SW_MX -> keyswitches:Kailh_socket_MX
Connections:
- net +5V: now also C4.1, C7.1, U29.16 (VCC), U7.16 (VCC)
- net C0: now also U7.14 (D0)
- net C1: now also U7.13 (D1)
- net C2: now also U7.12 (D2)
- net C3: now also U7.11 (D3)
- net C4: now also U29.14 (D0)
- net C5: now also U29.13 (D1)
- net C6: now also U29.12 (D2)
- net C7: now also U29.11 (D3)
- net GND: now also C4.2, C7.2, U29.15 (Mr), U29.2 (Oe2), U29.8 (GND), U7.15 (Mr), U7.2 (Oe2), U7.8 (GND)
- net L0: now also U7.3 (Q0)
- net L1: now also U7.4 (Q1)
- net L2: now also U7.5 (Q2)
- net L3: now also U7.6 (Q3)
- net L4: now also U29.3 (Q0)
- net L5: now also U29.4 (Q1)
- net L6: now also U29.5 (Q2)
- net L7: now also U29.6 (Q3)
- net LATCH_WEb: now also U29.10 (E2), U7.10 (E2)
- net Rb: now also U29.1 (Oe1), U29.9 (E1), U7.1 (Oe1), U7.9 (E1)
- new net ROW_CLK: U29.7 (Cp), U7.7 (Cp)
