File: Punchcard_Reader/Punchcard_Reader.kicad_sch (KiCad schematic)
At the start: 0 parts

Commit message: Added initial parts
Parts:
- added C11, C12: 0.1uF, Capacitor_SMD:C_0805_2012Metric_Pad1.18x1.45mm_HandSolder, symbol Device:C
- added D11: LED_BACKLIGHT, LED_THT:LED_D3.0mm, symbol Device:LED
- added R11: 120Ω, Resistor_SMD:R_0805_2012Metric_Pad1.20x1.40mm_HandSolder, symbol Device:R
- added U1, U2: 74HC14, Package_SO:SOIC-14_3.9x8.7mm_P1.27mm, symbol 74xx:74HC14
Connections:
- new net: D11.2 (A), R11.2
- new net +5V: C11.1, C12.1, R11.1, U1.14 (VCC), U2.14 (VCC)
- new net GND: C11.2, C12.2, D11.1 (K), U1.7 (GND), U2.11, U2.13, U2.7 (GND)
- no-connect marks 0 -> 2
Other:
- added sheet SensorBit0 (filtered_photodiode.kicad_sch)
- added sheet SensorBit1 (filtered_photodiode.kicad_sch)
- added sheet SensorBit2 (filtered_photodiode.kicad_sch)
- added sheet SensorBit3 (filtered_photodiode.kicad_sch)
- added sheet SensorBit4 (filtered_photodiode.kicad_sch)
- added sheet SensorBit5 (filtered_photodiode.kicad_sch)
- added sheet SensorBit6 (filtered_photodiode.kicad_sch)
- added sheet SensorBit7 (filtered_photodiode.kicad_sch)
- added sheet SensorClk (filtered_photodiode.kicad_sch)
- added sheet SensorClkSuppress (filtered_photodiode.kicad_sch)
